Commit message: adding CameraReader.h and CameraReader.cpp and writing out the logic for these sections

File: src/turtlebot3_simulations/turtlebot3_gazebo/urdf/turtlebot3_burger.urdf (robot description, URDF)
Before this commit: robot turtlebot3_burger, 7 links, 6 joints
Links:
- added link camera_link, mass 0.1; visual box size=0.05 0.05 0.05
Joints:
- added joint camera_joint: type fixed, parent base_link, child camera_link, origin xyz=0 0 0.1 rpy=0 0 0
